File: Crystal_hw/Crystal.kicad_pcb (KiCad board)
At the start: 2 copper layers, 77 x 77 mm, 71 parts, among them Q1 LED_5050, Q2 LED_5050, Q3 LED_5050, Q4 LED_5050, Q5 2N7002, SW1 BUTTON, SW2 BUTTON, SW3 BUTTON

Commit message: PCB is ready
Parts:
- added SA1: SS9, BtnsSwitches:SW_SS9, B.Cu at (163.4, 113.4)
- ANT1: footprint Antennas:Locket5 -> Antennas:Locket5_MIRR
- Logo1, RP3, RP4, XL1: moved to B.Cu
- SW1, SW2, SW3: value BUTTON -> IT1198; footprint BtnsSwitches:BTN_4x4_SMD -> BtnsSwitches:BTN_IT1198
- moved L1 155.8 mm to (109.6, 87.7), turned to 180 degrees
- moved BLN1 148.4 mm to (113.8, 87.0), turned to 180 degrees
- moved C4 144.5 mm to (118.2, 77.9), turned to 180 degrees
- moved R8 139.6 mm to (136.8, 98.8), turned to 180 degrees
- moved C13 139.2 mm to (119.5, 92.6), turned to -90 degrees
- moved C7 136.8 mm to (121.1, 92.6), turned to -90 degrees
- moved R3 134.2 mm to (117.9, 92.6), turned to -90 degrees
- moved R5 131.0 mm to (125.6, 102.8), turned to -90 degrees
- moved R6 130.3 mm to (136.8, 100.4), turned to 180 degrees
- moved XL3 129.6 mm to (133.2, 138.7)
- moved C2 129.0 mm to (110.1, 86.1), turned to 90 degrees
- moved C1 128.0 mm to (111.7, 87.7), turned to 180 degrees
- moved C3 127.8 mm to (109.1, 89.3), turned to -90 degrees
- moved L3 126.7 mm to (138.4, 96.0), turned to 90 degrees
- moved SW1 122.3 mm to (131.9, 70.5), turned to 180 degrees
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Connections:
- SW2 pad 1: /BTN_L -> +3v3
- SW2 pad 2: +3v3 -> /BTN_L
- SW3 pad 1: /BTN_R -> +3v3
- SW3 pad 2: +3v3 -> /BTN_R
- XL3 pad 2: +BATT -> /BAT2SW
Routing:
- net GND: track 0.00 -> 313.7 mm, vias 0 -> 254
- net +3v3: track 0.00 -> 134.7 mm, vias 0 -> 10
- net VCC: track 0.00 -> 60.2 mm, vias 0 -> 7
- net /BAT2SW: track 0.00 -> 35.4 mm
- net /CC_GDO0: track 0.00 -> 35.1 mm, vias 0 -> 2
- net /CC_GDO2: track 0.00 -> 34.8 mm, vias 0 -> 3
- net /CC_CS: track 0.00 -> 33.2 mm, vias 0 -> 2
- net /B3: track 0.00 -> 33.2 mm, vias 0 -> 2
- net /G3: track 0.00 -> 31.2 mm, vias 0 -> 2
- net /CC_MOSI: track 0.00 -> 29.5 mm, vias 0 -> 2
- net /R3: track 0.00 -> 29.4 mm, vias 0 -> 2
- net /CC_MISO: track 0.00 -> 29.1 mm, vias 0 -> 2
- net /CC_SCK: track 0.00 -> 28.2 mm, vias 0 -> 2
- net /ADC_BAT_EN: track 0.00 -> 27.3 mm, vias 0 -> 2
- net /BTN_PWR: track 0.00 -> 26.8 mm
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- added copper zone on B.Cu, net GND
- added copper zone on F.Cu, net GND
Other:
- board text added: "+"
- board text added: "-"
- board text added: "1"
- board text added: "GDO0"
- board text added: "GDO2"
- board text added: "ON"
- board text added: "Off"
- board text added: "Ostranna Crystal 1.0"
